File: LiquidLevelSensor/CAD/levelsensor/levelsensor.kicad_sch (KiCad schematic)
At the start: 5 parts, among them J1 Analog, J2 Digital, J3 Conn_01x02_Male

Commit message: updated drawing
Parts:
- added D1: LED, symbol Device:LED
- added R3: 1k, Resistor_SMD:R_0805_2012Metric_Pad1.20x1.40mm_HandSolder, symbol Device:R_US
- J3: footprint (none) -> Connector_Molex:Molex_SL_171971-0002_1x02_P2.54mm_Vertical
Connections:
- net D4: now also R3.1
- net GND: now also D1.1 (K)
- new net: D1.2 (A), R3.2
Changed lines of the file:
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@@
   (junction (at 161.29 81.28) (diameter 0) (color 0 0 0 0)
   )
+  (junction (at 149.86 73.66) (diameter 0) (color 0 0 0 0)
+  )
+  (junction (at 137.16 73.66) (diameter 0) (color 0 0 0 0)
+  )
   (junction (at 160.02 83.82) (diameter 0) (color 0 0 0 0)
   )
+  (junction (at 118.11 96.52) (diameter 0) (color 0 0 0 0)
+  )
   (wire (pts (xy 115.57 91.44) (xy 130.81 91.44))
     (stroke (width 0) (type solid) (color 0 0 0 0))
@@
     (stroke (width 0) (type default) (color 0 0 0 0))
   )
+  (wire (pts (xy 137.16 72.39) (xy 137.16 73.66))
+    (stroke (width 0) (type default) (color 0 0 0 0))
+  )
   (wire (pts (xy 77.47 71.12) (xy 95.25 71.12))
     (stroke (width 0) (type solid) (color 0 0 0 0))
@@
     (stroke (width 0) (type solid) (color 0 0 0 0))
   )
+  (wire (pts (xy 134.62 78.74) (xy 134.62 73.66))
+    (stroke (width 0) (type default) (color 0 0 0 0))
+  )
   (wire (pts (xy 115.57 71.12) (xy 130.81 71.12))
     (stroke (width 0) (type solid) (color 0 0 0 0))
@@
     (stroke (width 0) (type default) (color 0 0 0 0))
   )
+  (wire (pts (xy 157.48 73.66) (xy 157.48 96.52))
+    (stroke (width 0) (type default) (color 0 0 0 0))
+  )
+  (wire (pts (xy 144.78 73.66) (xy 149.86 73.66))
+    (stroke (width 0) (type default) (color 0 0 0 0))
+  )
+  (wire (pts (xy 157.48 96.52) (xy 118.11 96.52))
+    (stroke (width 0) (type default) (color 0 0 0 0))
+  )
   (wire (pts (xy 77.47 63.5) (xy 95.25 63.5))
     (stroke (width 0) (type solid) (color 0 0 0 0))
@@
     (stroke (width 0) (type solid) (color 0 0 0 0))
   )
+  (wire (pts (xy 149.86 73.66) (xy 151.13 73.66))
+    (stroke (width 0) (type default) (color 0 0 0 0))
+  )
   (wire (pts (xy 115.57 58.42) (xy 130.81 58.42))
     (stroke (width 0) (type solid) (color 0 0 0 0))
@@
     (stroke (width 0) (type solid) (color 0 0 0 0))
   )
-  (wire (pts (xy 115.57 78.74) (xy 130.81 78.74))
-    (stroke (width 0) (type solid) (color 0 0 0 0))
+  (wire (pts (xy 115.57 78.74) (xy 134.62 78.74))
+    (stroke (width 0) (type solid) (color 0 0 0 0))
+  )
+  (wire (pts (xy 134.62 73.66) (xy 137.16 73.66))
+    (stroke (width 0) (type default) (color 0 0 0 0))
   )
   (wire (pts (xy 161.29 110.49) (xy 74.93 110.49))
@@
       (effects (font (size 1.27 1.27)) (justify right) hide)
     )
-    (property "Footprint" "" (id 2) (at 171.45 81.28 0)
+    (property "Footprint" "Connector_Molex:Molex_SL_171971-0002_1x02_P2.54mm_Vertical" (id 2) (at 171.45 81.28 0)
       (effects (font (size 1.27 1.27)) hide)
     )
@@
     (pin "1")
   )
+  (symbol (lib_id "Device:LED") (at 153.67 73.66 180) (unit 1)
+    (in_bom yes) (on_board yes) (fields_autoplaced)
+    (property "Reference" "D1" (id 0) (at 155.2575 66.04 0))
+    (property "Value" "LED" (id 1) (at 155.2575 68.58 0))
+    (property "Footprint" "" (id 2) (at 153.67 73.66 0)
+      (effects (font (size 1.27 1.27)) hide)
+    )
+    (property "Datasheet" "~" (id 3) (at 153.67 73.66 0)
+      (effects (font (size 1.27 1.27)) hide)
+    )
+    (pin "1")
+    (pin "2")
+  )
   (symbol (lib_id "power:GND") (at 118.11 96.52 0) (unit 1)
     (in_bom yes) (on_board yes)
@@
   )
   (symbol (lib_id "Device:R_US") (at 143.51 81.28 90) (unit 1)
-    (in_bom yes) (on_board yes) (fields_autoplaced)
-    (property "Reference" "R1" (id 0) (at 143.51 74.93 90))
-    (property "Value" "12k" (id 1) (at 143.51 77.47 90))
+    (in_bom yes) (on_board yes)
+    (property "Reference" "R1" (id 0) (at 138.43 80.01 90))
+    (property "Value" "12k" (id 1) (at 149.86 80.01 90))
     (property "Footprint" "Resistor_SMD:R_0805_2012Metric_Pad1.20x1.40mm_HandSolder" (id 2) (at 143.764 80.264 90)
       (effects (font (size 1.27 1.27)) hide)
     )
     (property "Datasheet" "~" (id 3) (at 143.51 81.28 0)
+      (effects (font (size 1.27 1.27)) hide)
+    )
+    (pin "1")
+    (pin "2")
+  )
+  (symbol (lib_id "Device:R_US") (at 140.97 73.66 90) (unit 1)
+    (in_bom yes) (on_board yes)
+    (property "Reference" "R3" (id 0) (at 137.16 69.85 90))
+    (property "Value" "1k" (id 1) (at 142.24 69.85 90))
+    (property "Footprint" "Resistor_SMD:R_0805_2012Metric_Pad1.20x1.40mm_HandSolder" (id 2) (at 141.224 72.644 90)
+      (effects (font (size 1.27 1.27)) hide)
+    )
+    (property "Datasheet" "~" (id 3) (at 140.97 73.66 0)
       (effects (font (size 1.27 1.27)) hide)
     )
@@
       (reference "#PWR0105") (unit 1) (value "GND") (footprint "")
     )
+    (path "/902e8c8d-ace6-4cfc-b8da-2fc010ce6add"
+      (reference "D1") (unit 1) (value "LED") (footprint "LED_THT:LED_D3.0mm")
+    )
     (path "/00000000-0000-0000-0000-000056d719df"
       (reference "J1") (unit 1) (value "Analog") (footprint "Connector_PinHeader_2.54mm:PinHeader_1x15_P2.54mm_Vertical")
@@
       (reference "R2") (unit 1) (value "12k") (footprint "Resistor_SMD:R_0805_2012Metric_Pad1.20x1.40mm_HandSolder")
     )
-  )
+    (path "/c1cc7ff4-dbff-4cea-9b20-1006d47c73a9"
+      (reference "R3") (unit 1) (value "1k") (footprint "Resistor_SMD:R_0805_2012Metric_Pad1.20x1.40mm_HandSolder")
+    )
+  )
